File: EDA/EDA/microBoSL.sch (KiCad schematic (older format))
At the start: 55 parts, among them J1 Conn_01x04, J10 MOTOR_OUT, J11 Conn_01x03, J12 Conn_01x03, J13 Conn_01x03, J2 Conn_01x03, J3 Conn_01x04, J4 BATTERY CONN, J5 Conn_01x03, J6 Conn_01x04, J7 MOTOR_OUT, J8 USB_B_Micro, J9 MOTOR_OUT, Q1 DMP2165UW, SW1 RST_JMPR, SW2 AYZ0103AGRLC, U1 MAX40203ANS, U10 TPS709A33DBVT, U2 MAX40203ANS, U3 ATmega328P-MMH, U4 ZXBM5210-S, U5 74HC126PW-Q100, U6 MCP7940N-xSN, U7 FT232RQ, U8 ZXBM5210-S, U9 ZXBM5210-S, Y1 8MHz, Y2 32.768 kHz

Commit message: fixed o-ring circuit
Parts:
- removed U1, U2: MAX40203ANS, Package_BGA:WLP-4_0.73x0.73mm_Layout2x2_P0.35mm_Ball0.22mm_Pad0.2mm_NSMD, symbol Analog_Switch:MAX40200ANS
- added D4: CUS08F30,H3F, Diode_SMD:D_SOD-323, symbol Device:D
- added Q2: DMP2165UW, Package_TO_SOT_SMD:SOT-323_SC-70, symbol microBoSL-rescue:DMP2165UW
- added R11: 10 kΩ, Resistor_SMD:R_0402_1005Metric, symbol Device:R
- added R12: 4.7 MΩ, Capacitor_SMD:C_0402_1005Metric, symbol Device:R
Connections:
- net GND: now also R12.1
- net USB_V: now also D4.2 (A), R11.2
- net VBAT: now also Q2.3 (D)
- net at U10.3 (IN): now also D4.1 (K), Q2.2 (S)
- new net: Q2.1 (G), R11.1, R12.2
Other:
- moved on the sheet: C1, U10
Changed lines of the file:
@@
 Sheet 1 1
 Title "microBoSL Board"
-Date "2021-06-24"
-Rev "0.2.2"
+Date "2021-06-25"
+Rev "0.2.3"
 Comp ""
 Comment1 ""
@@
 	1    0    0    -1
 $EndComp
-Text GLabel 3750 3925 2    60   Input ~ 0
+Text GLabel 3775 3600 2    60   Input ~ 0
 V_3.3
 Text GLabel 1700 7050 0    60   Input ~ 0
@@
 L power:GND #PWR013
 U 1 1 5CEFF41F
-P 3475 4225
-F 0 "#PWR013" H 3475 3975 50  0001 C CNN
-F 1 "GND" H 3475 4075 50  0000 C CNN
-F 2 "" H 3475 4225 50  0000 C CNN
-F 3 "" H 3475 4225 50  0000 C CNN
-	1    3475 4225
+P 3500 3900
+F 0 "#PWR013" H 3500 3650 50  0001 C CNN
+F 1 "GND" H 3500 3750 50  0000 C CNN
+F 2 "" H 3500 3900 50  0000 C CNN
+F 3 "" H 3500 3900 50  0000 C CNN
+	1    3500 3900
 	1    0    0    -1
 $EndComp
@@
 Text Notes 475  2525 0    60   ~ 0
 3.3V Voltage Regulation\n
-Text Notes 525  5375 0    60   ~ 0
+Text Notes 550  5700 0    60   ~ 0
 Peripheral Connectivity
 Text GLabel 13325 1075 1    60   Input ~ 0
@@
 	1    0    0    -1
 $EndComp
-Wire Wire Line
-	1125 4425 1175 4425
-$Comp
-L power:GND #PWR03
-U 1 1 5FD837FD
-P 1625 4825
-F 0 "#PWR03" H 1625 4575 50  0001 C CNN
-F 1 "GND" H 1630 4652 50  0000 C CNN
-F 2 "" H 1625 4825 50  0001 C CNN
-F 3 "" H 1625 4825 50  0001 C CNN
-	1    1625 4825
-	1    0    0    -1
-$EndComp
-Text GLabel 1125 3475 0    60   Input ~ 0
+Text GLabel 975  3150 0    60   Input ~ 0
 USB_V
-Wire Wire Line
-	2025 4425 2125 4425
-Wire Wire Line
-	2025 3475 2125 3475
-Wire Wire Line
-	1125 3475 1175 3475
-$Comp
-L power:GND #PWR02
-U 1 1 5FD9A05F
-P 1625 3875
-F 0 "#PWR02" H 1625 3625 50  0001 C CNN
-F 1 "GND" H 1750 3750 50  0000 C CNN
-F 2 "" H 1625 3875 50  0001 C CNN
-F 3 "" H 1625 3875 50  0001 C CNN
-	1    1625 3875
-	1    0    0    -1
-$EndComp
 $Comp
 L Device:Crystal_GND24 Y1
@@
 USB_V
 Wire Notes Line
-	500  5250 4550 5250
+	525  5575 4575 5575
 Wire Notes Line
 	8050 1800 8050 500
@@
 L Device:C C1
 U 1 1 60874B04
-P 3475 4075
-F 0 "C1" H 3500 4175 50  0000 L CNN
-F 1 "2.2 μF" H 3500 3975 50  0000 L CNN
-F 2 "Capacitor_SMD:C_0805_2012Metric" H 3513 3925 50  0001 C CNN
-F 3 "https://au.mouser.com/datasheet/2/585/MLCC-1837944.pdf" H 3475 4075 50  0001 C CNN
-F 4 "https://au.mouser.com/ProductDetail/Samsung-Electro-Mechanics/CL21A225KAFNNNE?qs=sGAEpiMZZMuMW9TJLBQkXpDxzuCsSowO2NtmGkulgUw=" H 3475 4075 50  0001 C CNN "Supplier"
-	1    3475 4075
-	1    0    0    -1
-$EndComp
-Connection ~ 3475 3925
+P 3500 3750
+F 0 "C1" H 3525 3850 50  0000 L CNN
+F 1 "2.2 μF" H 3525 3650 50  0000 L CNN
+F 2 "Capacitor_SMD:C_0805_2012Metric" H 3538 3600 50  0001 C CNN
+F 3 "https://au.mouser.com/datasheet/2/585/MLCC-1837944.pdf" H 3500 3750 50  0001 C CNN
+F 4 "https://au.mouser.com/ProductDetail/Samsung-Electro-Mechanics/CL21A225KAFNNNE?qs=sGAEpiMZZMuMW9TJLBQkXpDxzuCsSowO2NtmGkulgUw=" H 3500 3750 50  0001 C CNN "Supplier"
+	1    3500 3750
+	1    0    0    -1
+$EndComp
+Connection ~ 3500 3600
 $Comp
 L Driver_Motor:ZXBM5210-S U4
@@
 	1    0    0    -1
 $EndComp
-Text GLabel 1125 4425 0    60   Input ~ 0
+Text GLabel 975  4100 0    60   Input ~ 0
 VBAT
 $Comp
@@
 NoConn ~ 14050 4575
 Wire Wire Line
-	3475 3925 3750 3925
+	3500 3600 3775 3600
 Text GLabel 3300 5975 0    60   Input ~ 0
 MOSI
@@
 L power:GND #PWR0103
 U 1 1 60D5075B
-P 2825 4325
-F 0 "#PWR0103" H 2825 4075 50  0001 C CNN
-F 1 "GND" H 2950 4200 50  0000 C CNN
-F 2 "" H 2825 4325 50  0001 C CNN
-F 3 "" H 2825 4325 50  0001 C CNN
-	1    2825 4325
+P 2850 4000
+F 0 "#PWR0103" H 2850 3750 50  0001 C CNN
+F 1 "GND" H 2975 3875 50  0000 C CNN
+F 2 "" H 2850 4000 50  0001 C CNN
+F 3 "" H 2850 4000 50  0001 C CNN
+	1    2850 4000
 	1    0    0    -1
 $EndComp
@@
 L microBoSL-rescue:TPS709A33DBVT U10
 U 1 1 60D50766
-P 2825 4025
-F 0 "U10" H 2575 4375 60  0000 C CNN
-F 1 "TPS709A33DBVT" H 2875 4275 60  0000 C CNN
-F 2 "Package_TO_SOT_SMD:SOT-23-5" H 2975 3975 60  0001 C CNN
-F 3 "https://www.ti.com/lit/ds/symlink/tps709.pdf?ts=1619152264234&ref_url=https%253A%252F%252Fau.mouser.com%252F" H 2975 3975 60  0001 C CNN
-F 4 "https://au.mouser.com/ProductDetail/Texas-Instruments/TPS709A33DBVT?qs=9yI11AV48ZQgL37ZcAbPUA==" H 2825 4025 50  0001 C CNN "Supplier"
-	1    2825 4025
-	1    0    0    -1
-$EndComp
-NoConn ~ 2425 4075
-Wire Wire Line
-	3225 3925 3475 3925
-Wire Wire Line
-	2125 3475 2125 3925
-Wire Wire Line
-	2125 3925 2425 3925
-Connection ~ 2125 3925
-$Comp
-L Analog_Switch:MAX40200ANS U1
-U 1 1 60D5BCF1
-P 1625 3575
-F 0 "U1" H 1625 3942 50  0000 C CNN
-F 1 "MAX40203ANS" H 1625 3851 50  0000 C CNN
-F 2 "Package_BGA:WLP-4_0.73x0.73mm_Layout2x2_P0.35mm_Ball0.22mm_Pad0.2mm_NSMD" H 1625 3975 50  0001 C CNN
-F 3 "https://datasheets.maximintegrated.com/en/ds/MAX40200.pdf" H 1625 3975 50  0001 C CNN
-	1    1625 3575
-	1    0    0    -1
-$EndComp
-$Comp
-L Analog_Switch:MAX40200ANS U2
-U 1 1 60D5C188
-P 1625 4525
-F 0 "U2" H 1625 4892 50  0000 C CNN
-F 1 "MAX40203ANS" H 1625 4801 50  0000 C CNN
-F 2 "Package_BGA:WLP-4_0.73x0.73mm_Layout2x2_P0.35mm_Ball0.22mm_Pad0.2mm_NSMD" H 1625 4925 50  0001 C CNN
-F 3 "https://datasheets.maximintegrated.com/en/ds/MAX40200.pdf" H 1625 4925 50  0001 C CNN
-	1    1625 4525
-	1    0    0    -1
-$EndComp
-Wire Wire Line
-	1175 3475 1175 3675
-Wire Wire Line
-	1175 3675 1225 3675
-Connection ~ 1175 3475
-Wire Wire Line
-	1175 3475 1225 3475
-Wire Wire Line
-	1175 4425 1175 4625
-Wire Wire Line
-	1175 4625 1225 4625
-Connection ~ 1175 4425
-Wire Wire Line
-	1175 4425 1225 4425
-Wire Wire Line
-	2125 3925 2125 4425
+P 2850 3700
+F 0 "U10" H 2600 4050 60  0000 C CNN
+F 1 "TPS709A33DBVT" H 2900 3950 60  0000 C CNN
+F 2 "Package_TO_SOT_SMD:SOT-23-5" H 3000 3650 60  0001 C CNN
+F 3 "https://www.ti.com/lit/ds/symlink/tps709.pdf?ts=1619152264234&ref_url=https%253A%252F%252Fau.mouser.com%252F" H 3000 3650 60  0001 C CNN
+F 4 "https://au.mouser.com/ProductDetail/Texas-Instruments/TPS709A33DBVT?qs=9yI11AV48ZQgL37ZcAbPUA==" H 2850 3700 50  0001 C CNN "Supplier"
+	1    2850 3700
+	1    0    0    -1
+$EndComp
+NoConn ~ 2450 3750
+Wire Wire Line
+	3250 3600 3500 3600
+Wire Wire Line
+	2150 3150 2150 3600
+Wire Wire Line
+	2150 3600 2450 3600
+Connection ~ 2150 3600
+Wire Wire Line
+	2150 3600 2150 4100
 $Comp
 L Connector_Generic:Conn_01x04 J6
@@
 Text Notes 4575 575  0    60   ~ 0
 MCU
+$Comp
+L Device:D D4
+U 1 1 60D5DB85
+P 1725 3150
+F 0 "D4" H 1725 2933 50  0000 C CNN
+F 1 "CUS08F30,H3F" H 1725 3024 50  0000 C CNN
+F 2 "Diode_SMD:D_SOD-323" H 1725 3150 50  0001 C CNN
+F 3 "https://au.mouser.com/datasheet/2/408/CUS08F30_datasheet_en_20140414-1916097.pdf" H 1725 3150 50  0001 C CNN
+F 4 "https://au.mouser.com/ProductDetail/Toshiba/CUS08F30H3F?qs=sGAEpiMZZMtbRapU8LlZD%252BCy%2FVT4IDP8xwNxSitleb9JD5GJ4tdDdA%3D%3D" H 1725 3025 50  0001 C CNN "Supplier"
+	1    1725 3150
+	-1   0    0    1
+$EndComp
+$Comp
+L microBoSL-rescue:DMP2165UW Q2
+U 1 1 60D5E861
+P 1725 4200
+F 0 "Q2" H 1930 4246 50  0000 L CNN
+F 1 "DMP2165UW" H 1930 4155 50  0000 L CNN
+F 2 "Package_TO_SOT_SMD:SOT-323_SC-70" H 1925 4300 50  0001 C CNN
+F 3 "https://au.mouser.com/datasheet/2/115/DMP2165UW-1365845.pdf" H 1725 4200 50  0001 C CNN
+F 4 "https://au.mouser.com/ProductDetail/Diodes-Incorporated/DMP2165UW-7?qs=y6ZabgHbY%252ByvCNbAJzQtdQ==" H 1725 4200 50  0001 C CNN "Supplier"
+	1    1725 4200
+	0    -1   -1   0
+$EndComp
+Wire Wire Line
+	975  4100 1525 4100
+Wire Wire Line
+	1925 4100 2150 4100
+$Comp
+L Device:R R11
+U 1 1 60D6FF18
+P 1400 4525
+F 0 "R11" V 1480 4525 50  0000 C CNN
+F 1 "10 kΩ" V 1300 4525 50  0000 C CNN
+F 2 "Resistor_SMD:R_0402_1005Metric" V 1330 4525 50  0001 C CNN
+F 3 "https://au.mouser.com/datasheet/2/427/crcwce3-1762584.pdf" H 1400 4525 50  0001 C CNN
+F 4 "https://au.mouser.com/ProductDetail/Vishay-Dale/CRCW040210K0FKEDC?qs=/ha2pyFaduiHT66YdUA2uA4sF2ipRtotJ1IZi2VsJbqIToNUmUEwdxElf6FK9FXM" H 1400 4525 50  0001 C CNN "Supplier"
+	1    1400 4525
+	0    1    1    0
+$EndComp
+$Comp
+L Device:R R12
+U 1 1 60D70459
+P 1725 4775
+F 0 "R12" H 1795 4821 50  0000 L CNN
+F 1 "4.7 MΩ" H 1400 4725 50  0000 L CNN
+F 2 "Capacitor_SMD:C_0402_1005Metric" V 1655 4775 50  0001 C CNN
+F 3 "https://au.mouser.com/datasheet/2/427/crcwce3-1762584.pdf" H 1725 4775 50  0001 C CNN
+F 4 "https://au.mouser.com/ProductDetail/Vishay-Dale/CRCW04024M70FKEDC?qs=/ha2pyFaduiHT66YdUA2uBTzMf/OTznJ3p5fz7SH86RaDbjs2LFbjBRRStKMxFDa" H 1725 4775 50  0001 C CNN "Supplier"
+	1    1725 4775
+	-1   0    0    1
+$EndComp
+$Comp
+L power:GND #PWR02
+U 1 1 60D8F248
+P 1725 5025
+F 0 "#PWR02" H 1725 4775 50  0001 C CNN
+F 1 "GND" H 1725 4875 50  0000 C CNN
+F 2 "" H 1725 5025 50  0000 C CNN
+F 3 "" H 1725 5025 50  0000 C CNN
+	1    1725 5025
+	1    0    0    -1
+$EndComp
+Wire Wire Line
+	1725 5025 1725 4925
+Wire Wire Line
+	1725 4400 1725 4525
+Wire Wire Line
+	1550 4525 1725 4525
+Connection ~ 1725 4525
+Wire Wire Line
+	1725 4525 1725 4625
+Wire Wire Line
+	1250 4525 1250 3150
+Wire Wire Line
+	1250 3150 1575 3150
+Wire Wire Line
+	1875 3150 2150 3150
+Wire Wire Line
+	1250 3150 975  3150
+Connection ~ 1250 3150
 $EndSCHEMATC

Commit message: rebase for adding wireless to microbosl
Parts:
- removed C12, C13, C14, C2, C3, C4, C7: 100 nF, Capacitor_SMD:C_0402_1005Metric, symbol Device:C
- removed D4: CUS08F30,H3F, Diode_SMD:D_SOD-323, symbol Device:D
- removed J10, J9: MOTOR_OUT, Connector_PinHeader_2.54mm:PinHeader_1x02_P2.54mm_Vertical, symbol Connector_Generic:Conn_01x02
- removed J11, J12, J13, J5: Conn_01x03, Connector_PinHeader_2.00mm:PinHeader_1x03_P2.00mm_Vertical, symbol Connector_Generic:Conn_01x03
- removed J2: Conn_01x03, Connector_PinHeader_1.27mm:PinHeader_1x03_P1.27mm_Vertical, symbol Connector_Generic:Conn_01x03
- removed J6: Conn_01x04, Connector_PinHeader_1.27mm:PinHeader_1x04_P1.27mm_Vertical, symbol Connector_Generic:Conn_01x04
- removed Q1, Q2: DMP2165UW, Package_TO_SOT_SMD:SOT-323_SC-70, symbol microBoSL-rescue:DMP2165UW
- removed R1, R11: 10 kΩ, Resistor_SMD:R_0402_1005Metric, symbol Device:R
- removed R12, R5, R6: 4.7 MΩ, Capacitor_SMD:C_0402_1005Metric, symbol Device:R
- removed SW2: AYZ0103AGRLC, SIMFootprints:AYZ0103AGRLC, symbol microBoSL-rescue:AYZ0103AGRLC
- removed U10: TPS709A33DBVT, Package_TO_SOT_SMD:SOT-23-5, symbol microBoSL-rescue:TPS709A33DBVT
- removed U3: ATmega328P-MMH, Package_DFN_QFN:QFN-28-1EP_4x4mm_P0.45mm_EP2.4x2.4mm, symbol MCU_Microchip_ATmega:ATmega328P-MMH
- removed U4, U8, U9: ZXBM5210-S, Package_SO:SOIC-8_3.9x4.9mm_P1.27mm, symbol Driver_Motor:ZXBM5210-S
- added J2: Conn_02x03_Odd_Even, Connector_PinHeader_2.54mm:PinHeader_2x03_P2.54mm_Vertical, symbol Connector_Generic:Conn_02x03_Odd_Even
- added J3: Conn_01x04, Connector_PinHeader_1.27mm:PinHeader_1x04_P1.27mm_Vertical, symbol Connector_Generic:Conn_01x04
- added J6: Conn_01x10, Connector_PinHeader_1.27mm:PinHeader_1x10_P1.27mm_Vertical, symbol Connector_Generic:Conn_01x10
- added Q1: DMG2302UK, Package_TO_SOT_SMD:SOT-23, symbol Device:Q_NMOS_GSD
- added R2: 1 kΩ, Resistor_SMD:R_0402_1005Metric, symbol Device:R
- added U1, U2: MAX40200ANS, Package_BGA:WLP-4_0.73x0.73mm_Layout2x2_P0.35mm_Ball0.22mm_Pad0.2mm_NSMD, symbol Analog_Switch:MAX40200ANS
- added U3: MCP1700-3302E_SOT23, Package_TO_SOT_SMD:SOT-23, symbol Regulator_Linear:MCP1700-3302E_SOT23
- added U4: ATmega328-MMH, Package_DFN_QFN:QFN-28-1EP_4x4mm_P0.45mm_EP2.4x2.4mm, symbol MCU_Microchip_ATmega:ATmega328-MMH
- C1: value 2.2 μF -> 1 μF; footprint Capacitor_SMD:C_0805_2012Metric -> Capacitor_SMD:C_1206_3216Metric; Supplier https://au.mouser.com/ProductDetail/Samsung-Electro-Mechani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 -> (none)
- C2: renamed from C6; value 15 pF -> 22 pF; Supplier https://au.mouser.com/ProductDetail/KEMET/C0402C150J8HACTU?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 -> (none)
- C3: renamed from C5; value 15 pF -> 22 pF; Supplier https://au.mouser.com/ProductDetail/KEMET/C0402C150J8HACTU?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 -> (none)
- C4: renamed from C9; value 15 pF -> 12 pF; Supplier https://au.mouser.com/ProductDetail/KEMET/C0402C150J8HACTU?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 -> (none)
- C5: renamed from C8; value 15 pF -> 12 pF; Supplier https://au.mouser.com/ProductDetail/KEMET/C0402C150J8HACTU?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 -> (none)
- C6: renamed from C10; footprint Capacitor_SMD:C_0402_1005Metric -> Capacitor_SMD:C_0603_1608Metric; Supplier https://au.mouser.com/ProductDetail/AVX/04026D104KAT2A?qs=s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 -> (none)
- C7: renamed from C11; footprint Capacitor_SMD:C_0402_1005Metric -> Capacitor_SMD:C_0603_1608Metric; Supplier https://au.mouser.com/ProductDetail/AVX/04026D104KAT2A?qs=s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 -> (none)
- D1: renamed from D2; Supplier https://au.mouser.com/ProductDetail/Wurth-Elektronik/150060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 -> (none)
- D2: renamed from D3; Supplier https://au.mouser.com/datasheet/2/445/150060YS55040-1714218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 -> (none)
- D3: renamed from D1; Supplier https://au.mouser.com/ProductDetail/Wurth-Elektronik/150060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 -> (none)
- J1: footprint Connector_PinHeader_1.27mm:PinHeader_1x04_P1.27mm_Vertical -> Connector_PinHeader_2.54mm:PinHeader_1x04_P2.54mm_Vertical
- J5: renamed from J4; value BATTERY CONN -> Conn_01x02
- J7: value MOTOR_OUT -> Conn_01x02
- J8: symbol microBoSL-rescue:USB_B_Micro-Connector -> Connector:USB_B_Micro; Supplier https://au.mouser.com/ProductDetail/Molex/105133-0001?qs=nm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 -> (none)
- R1: renamed from R2; Supplier https://au.mouser.com/ProductDetail/Vishay-Dale/CRCW040210K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 -> (none)
- R3: renamed from R4; Supplier https://au.mouser.com/ProductDetail/Vishay-Dale/CRCW040210K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 -> (none)
- R4: renamed from R3; Supplier https://au.mouser.com/ProductDetail/Vishay-Dale/CRCW040210K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 -> (none)
- R5: renamed from R7; Supplier https://au.mouser.com/ProductDetail/Vishay-Dale/CRCW040210K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 -> (none)
- R6: renamed from R8; Supplier https://au.mouser.com/ProductDetail/Vishay-Dale/CRCW04023K3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 -> (none)
- R7: renamed from R9; Supplier https://au.mouser.com/ProductDetail/Vishay-Dale/CRCW04023K3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 -> (none)
- R8: renamed from R10; Supplier https://au.mouser.com/ProductDetail/Vishay-Dale/CRCW04023K3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 -> (none)
- SW1: value RST_JMPR -> PTS636 SM43J SMTR LFS; footprint Jumper:SolderJumper-2_P1.3mm_Open_RoundedPad1.0x1.5mm -> SIMFootprints:PTS636 SM43J SMTR LFS
- U5: renamed from U6; Supplier https://www.digikey.com.au/product-detail/en/MCP7940NT-I-MN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 -> (none)
- U6: renamed from U5; Supplier https://au.mouser.com/ProductDetail/Nexperia/74HC126PW-Q100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 -> (none)
- U7: Supplier https://au.mouser.com/ProductDetail/FTDI/FT232RQ-REEL?qs=D1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 -> (none)
- Y1: footprint Crystal:Crystal_SMD_5032-4Pin_5.0x3.2mm -> Crystal:Crystal_SMD_EuroQuartz_MT-4Pin_3.2x2.5mm; Supplier https://au.mouser.com/ProductDetail/Diodes-Incorporated/F90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 -> (none)
- Y2: footprint Crystal:Crystal_SMD_2012-2Pin_2.0x1.2mm -> Crystal:Crystal_SMD_EuroQuartz_EQ161-2Pin_3.2x1.5mm; Supplier https://au.mouser.com/ProductDetail/IQD/LFXTAL050789Reel?qs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 -> (none)
- renumbered J3 to J4
Connections:
- net VBAT is gone; now on net VPP: J4.2 (Pin_2)
- net AREF: now also U4.17 (AREF)
- net GND: now also J7.2 (Pin_2), U5.3 (VBAT), J2.1 (Pin_1), J2.2 (Pin_2), J3.1 (Pin_1), Q1.2 (S), R2.1, U1.B2 (GND), U2.B2 (GND), U3.1 (GND), U4.18 (GND), U4.29 (GND), U4.4 (GND)
- net Hall_WKE_S: now also J2.5 (Pin_5), U4.21 (PC2)
- net RTC_I: now also U4.28 (PD2)
- net SCL: now also U4.24 (PC5)
- net SDA: now also U4.23 (PC4)
- net TLL_RST: now also J3.2 (Pin_2), U4.25 (~RESET~/PC6)
- net TLL_RX: now also J3.3 (Pin_3), U4.26 (PD0)
- net TLL_TX: now also J3.4 (Pin_4), U4.27 (PD1)
- net USB_V: now also U1.A1 (VDD), U1.B1 (EN)
- net VPP: now also U2.A1 (VDD), U2.B1 (EN)
- net V_3.3: now also U3.2 (VO), U4.16 (AVCC), U4.3 (VCC)
- net at C2.2, Y1.1: now also U4.6 (XTAL2/PB7)
- net at C3.2, Y1.3: now also U4.5 (XTAL1/PB6)
- net at J7.1 (Pin_1): now also Q1.3 (D)
- new net: U1.A2 (OUT), U2.A2 (OUT), U3.3 (VI)
- new net A1: J6.9 (Pin_9), U4.20 (PC1)
- new net A3: J6.10 (Pin_10), U4.22 (PC3)
- new net D10: J6.5 (Pin_5), U4.12 (PB2)
- new net D11: J6.6 (Pin_6), U4.13 (PB3)
- new net D12: J6.7 (Pin_7), U4.14 (PB4)
- new net D13: J6.8 (Pin_8), U4.15 (PB5)
- new net D3: J6.1 (Pin_1), U4.1 (PD3)
- new net D4: J6.2 (Pin_2), U4.2 (PD4)
- new net D7: J6.3 (Pin_3), U4.9 (PD7)
- new net D8: J6.4 (Pin_4), U4.10 (PB0)
- new net Hall_CNT_P: J2.4 (Pin_4), U4.8 (PD6)
- new net Hall_CNT_S: J2.6 (Pin_6), U4.19 (PC0)
- new net Hall_WKE_P: J2.3 (Pin_3), U4.7 (PD5)
- new net MOSFET: Q1.1 (G), R2.2, U4.11 (PB1)
- no-connect marks 18 -> 15
Other:
- note added: "Hall Count"
- note added: "Motor MOSFET"
- note removed: "Battery Switch"
- note removed: "Motor H Bridges"
- moved on the sheet: C2, C3, C4, C5, C6, C7, D1, D2, D3, J1, J4, J5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
