File: EDA/EDA/microBoSL.kicad_sch (KiCad schematic)
At the start: 65 parts, among them J1 Conn_01x04, J2 Conn_01x03, J3 Conn_01x04, J4 Conn_01x04, J5 Conn_01x02, J8 USB_B_Micro, J9 MOTOR_OUT, Q1 DMP2165UW, Q2 DMP2165UW, U1 TPS709A33DBVT, U2 ZXBM5210-S, U4 ATmega328-MMH, U6 74HC126PW-Q100, U7 FT232RQ, U8 Si4463, Y1 8MHz, Y2 32.768 kHz, Y3 30 MHz

Commit message: added BOM and finished most layout
Parts:
- AE1: value Antenna -> (none); footprint Connector_PinHeader_2.54mm:PinHeader_1x01_P2.54mm_Vertical -> (none)
- C1: value 2.2 μF -> (none); footprint Capacitor_SMD:C_0805_2012Metric -> (none)
- C10, C12: value 5.1 pF -> (none); footprint Capacitor_SMD:C_0402_1005Metric -> (none); Supplier (none) -> https://au.mouser.com/ProductDetail/KEMET/CBR04C519C5GAC?qs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
- C11: value 6.8 pF -> (none); footprint Capacitor_SMD:C_0402_1005Metric -> (none); Supplier (none) -> https://au.mouser.com/ProductDetail/KEMET/C0402C689C5HACTU?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
- C13: value 12 pF -> (none); footprint Capacitor_SMD:C_0402_1005Metric -> (none); Supplier (none) -> https://au.mouser.com/ProductDetail/KEMET/C0402C120J5HACTU?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
- C14: value 18 pF -> (none); footprint Capacitor_SMD:C_0402_1005Metric -> (none); Supplier (none) -> https://au.mouser.com/ProductDetail/KEMET/C0402C180J5GAC?qs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
- C15: value 9.1 pF -> (none); footprint Capacitor_SMD:C_0402_1005Metric -> (none); Supplier (none) -> https://au.mouser.com/ProductDetail/KEMET/CBR04C919B5GAC?qs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
- C16, C4, C5: value 100 nF -> (none); footprint Capacitor_SMD:C_0402_1005Metric -> (none); Supplier https://au.mouser.com/ProductDetail/AVX/04026D104KAT2A?qs=s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 -> https://au.mouser.com/ProductDetail/KEMET/C0402C103K3RACTU?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
- C17, C18: value 15 pF -> (none); footprint Capacitor_SMD:C_0402_1005Metric -> (none); Supplier https://au.mouser.com/ProductDetail/KEMET/C0402C150J8HACTU?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 -> https://au.mouser.com/ProductDetail/KEMET/C0402C150J4GACAUT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
- C2, C3: value 22 pF -> (none); footprint Capacitor_SMD:C_0402_1005Metric -> (none); Supplier (none) -> https://au.mouser.com/ProductDetail/KEMET/C0402C220J8HACTU?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
- C6, C7: value 100 nF -> (none); footprint Capacitor_SMD:C_0603_1608Metric -> (none); Supplier (none) -> https://au.mouser.com/ProductDetail/KEMET/C0402C103K3RACTU?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
- C8: value 100 pF -> (none); footprint Capacitor_SMD:C_0402_1005Metric -> (none); Supplier (none) -> https://au.mouser.com/ProductDetail/KEMET/C0402C101K3RACAUT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
- C9: value 100 nF -> (none); footprint Capacitor_SMD:C_0402_1005Metric -> (none); Supplier (none) -> https://au.mouser.com/ProductDetail/KEMET/C0402C103K3RACTU?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
- D1, D2, D3: value LED -> (none); footprint LED_SMD:LED_0603_1608Metric -> (none); Supplier (none) -> https://au.mouser.com/ProductDetail/Wurth-Elektronik/150060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
- D4: value CUS08F30,H3F -> (none); footprint Diode_SMD:D_SOD-323 -> (none)
- F1: Supplier (none) -> https://au.element14.com/bel-fuse/0685t1000-01/fuse-smd-1a-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; URL https://au.element14.com/bel-fuse/0685t1000-01/fuse-smd-1a-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 -> (none)
- J1, J4: value Conn_01x04 -> (none); footprint Connector_PinHeader_2.54mm:PinHeader_1x04_P2.54mm_Vertical -> (none)
- J2: value Conn_01x03 -> (none); footprint Connector_PinHeader_2.54mm:PinHeader_1x03_P2.54mm_Vertical -> (none)
- J3: value Conn_01x04 -> (none); footprint Connector_PinHeader_1.27mm:PinHeader_1x04_P1.27mm_Vertical -> (none)
- J5: value Conn_01x02 -> (none); footprint Connector_PinHeader_2.54mm:PinHeader_1x02_P2.54mm_Vertical -> (none)
- J8: value USB_B_Micro -> (none); footprint Connector_USB:USB_Micro-B_Molex-105133-0001 -> (none); Supplier (none) -> https://au.mouser.com/ProductDetail/Molex/105133-0001?qs=nm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
- J9: value MOTOR_OUT -> (none); footprint Connector_PinHeader_2.54mm:PinHeader_1x02_P2.54mm_Vertical -> (none)
- L1: value 220 nH -> (none); footprint Inductor_SMD:L_0402_1005Metric -> (none); Supplier (none) -> https://au.mouser.com/ProductDetail/Wurth-Elektronik/744784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
- L2: value 68 nH -> (none); footprint Inductor_SMD:L_0402_1005Metric -> (none); Supplier (none) -> https://au.mouser.com/ProductDetail/Wurth-Elektronik/784780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
- L3: value 24 nH -> (none); footprint Inductor_SMD:L_0402_1005Metric -> (none); Supplier (none) -> https://au.mouser.com/ProductDetail/Murata-Electronics/LQW1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
- L4: value 27 nH -> (none); footprint Inductor_SMD:L_0402_1005Metric -> (none); Supplier (none) -> https://au.mouser.com/ProductDetail/Wurth-Elektronik/784780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
- L5, L6: value 12 nH -> (none); footprint Inductor_SMD:L_0402_1005Metric -> (none); Supplier (none) -> https://au.mouser.com/ProductDetail/Wurth-Elektronik/744784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
- Q1, Q2: value DMP2165UW -> (none); footprint Package_TO_SOT_SMD:SOT-323_SC-70 -> (none)
- R1, R5: value 10 kΩ -> (none); footprint Resistor_SMD:R_0402_1005Metric -> (none); Supplier (none) -> https://au.mouser.com/ProductDetail/Panasonic/ERJ-2RKF1002X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
- R10, R2, R3, R9: value 10 kΩ -> (none); footprint Resistor_SMD:R_0402_1005Metric -> (none); Supplier https://au.mouser.com/ProductDetail/Vishay-Dale/CRCW040210K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 -> https://au.mouser.com/ProductDetail/Panasonic/ERJ-2RKF1002X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
- R11, R12, R4: value 4.7 MΩ -> (none); footprint Capacitor_SMD:C_0402_1005Metric -> (none)
- R6, R7, R8: value 3.3 kΩ -> (none); footprint Resistor_SMD:R_0402_1005Metric -> (none); Supplier (none) -> https://au.mouser.com/ProductDetail/Panasonic/ERJ-2GEJ332X?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
- U1: value TPS709A33DBVT -> (none); footprint Package_TO_SOT_SMD:SOT-23-5 -> (none)
- U2: value ZXBM5210-S -> (none); footprint Package_SO:SOIC-8_3.9x4.9mm_P1.27mm -> (none)
- U3: Supplier (none) -> https://au.mouser.com/ProductDetail/Microchip-Technology/MC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
- U4: value ATmega328-MMH -> (none); footprint Package_DFN_QFN:QFN-28-1EP_4x4mm_P0.45mm_EP2.4x2.4mm -> (none); Supplier (none) -> https://au.mouser.com/ProductDetail/Microchip-Technology-At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
- U6: value 74HC126PW-Q100 -> (none); footprint Package_SO:TSSOP-14_4.4x5mm_P0.65mm -> (none); Supplier (none) -> https://au.mouser.com/ProductDetail/Nexperia/74HC126PW-Q100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
- U7: value FT232RQ -> (none); footprint Package_DFN_QFN:QFN-32-1EP_5x5mm_P0.5mm_EP3.1x3.1mm -> (none); Supplier (none) -> https://au.mouser.com/ProductDetail/FTDI/FT232RQ-REEL?qs=D1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
- U8: value Si4463 -> (none); footprint Package_DFN_QFN:QFN-20-1EP_4x4mm_P0.5mm_EP2.6x2.6mm_ThermalVias -> (none); Supplier (none) -> https://au.mouser.com/ProductDetail/Silicon-Labs/SI4463-C2A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
- Y1: value 8MHz -> (none); footprint Crystal:Crystal_SMD_EuroQuartz_MT-4Pin_3.2x2.5mm -> (none); Supplier (none) -> https://au.mouser.com/ProductDetail/ECS/ECS-80-18-33-JGN-TR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
- Y2: value 32.768 kHz -> (none); footprint Crystal:Crystal_SMD_2012-2Pin_2.0x1.2mm -> (none)
- Y3: value 30 MHz -> (none); footprint Crystal:Crystal_SMD_Abracon_ABM8G-4Pin_3.2x2.5mm -> (none); Supplier (none) -> https://au.mouser.com/ProductDetail/ABRACON/ABM8AIG-30.000M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
